File: PCB/projects.kicad_pcb (KiCad board)
At the start: 2 copper layers, 61.9 x 43.7 mm, 7 parts, among them SW1 SW_Push, SW2 SW_Push, SW3 SW_Push, SW4 SW_Push, U1 XIAO-RP2040-DIP

Commit message: Add files via upload
Parts:
- added J1: Conn_01x04, OLED:SSD1306-0.91-OLED-4pin-128x32, F.Cu at (108.4, 87.7)
- moved U1 1.82 mm to (89.2, 58.6)
Connections:
- U1 pad 6: unconnected-(U1-GPIO7/SCL-Pad6) -> Net-(J1-Pin_3)
- U1 pad 7: unconnected-(U1-GPIO0/TX-Pad7) -> Net-(J1-Pin_4)
Routing:
- net Net-(J1-Pin_4): track 0.00 -> 42.9 mm
- net Net-(J1-Pin_3): track 0.00 -> 39.3 mm
- net Net-(U1-GPIO2/SCK): track 61.6 -> 98.4 mm
- net GND: track 149.6 -> 134.1 mm
- net +5V: track 52.6 -> 67.1 mm
- net Net-(U1-GPIO1/RX): track 36.9 -> 45.0 mm
- net Net-(U1-GPIO4/MISO): track 30.2 -> 37.5 mm
- net Net-(U1-GPIO3/MOSI): track 21.3 -> 18.7 mm
- net Net-(D1-DIN): track 30.7 -> 29.2 mm
Other:
- board size 61.9 x 43.7 mm -> 73.8 x 42.5 mm
